File: door-sign/door-sign.kicad_sch (KiCad schematic)
At the start: 3 parts, among them SW1 200MSP1T1B1M2QEH

Commit message: components done
Parts:
- added D1, D2: WP813GD, parts:LEDRD254W57D1100H1450, symbol parts:WP813GD
- added R2, R3: CF12JT220R, parts:STA_CF12_STP, symbol parts:CF12JT220R
Changed lines of the file:
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@@
+    )
+  )
+  (symbol (lib_id "parts:WP813GD") (at 201.93 83.82 0) (unit 1)
+    (in_bom yes) (on_board yes) (dnp no) (fields_autoplaced)
+    (property "Reference" "D1" (at 200.66 74.93 0)
+      (effects (font (size 1.27 1.27)))
+    )
+    (property "Value" "WP813GD" (at 200.66 77.47 0)
+      (effects (font (size 1.27 1.27)))
+    )
+    (property "Footprint" "parts:LEDRD254W57D1100H1450" (at 201.93 83.82 0)
+      (effects (font (size 1.27 1.27)) (justify bottom) hide)
+    )
+    (property "Datasheet" "" (at 201.93 83.82 0)
+      (effects (font (size 1.27 1.27)) hide)
+    )
+    (property "PARTREV" "V.9B" (at 201.93 83.82 0)
+      (effects (font (size 1.27 1.27)) (justify bottom) hide)
+    )
+    (property "STANDARD" "IPC 7351B" (at 201.93 83.82 0)
+      (effects (font (size 1.27 1.27)) (justify bottom) hide)
+    )
+    (property "SNAPEDA_PACKAGE_ID" "41838" (at 201.93 83.82 0)
+      (effects (font (size 1.27 1.27)) (justify bottom) hide)
+    )
+    (property "MAXIMUM_PACKAGE_HEIGHT" "14.5 mm" (at 201.93 83.82 0)
+      (effects (font (size 1.27 1.27)) (justify bottom) hide)
+    )
+    (property "MANUFACTURER" "Kingbright" (at 201.93 83.82 0)
+      (effects (font (size 1.27 1.27)) (justify bottom) hide)
+    )
+    (pin "1")
+    (pin "2")
+    (instances
+      (project "door-sign"
+        (path "/e88230cd-1344-4912-a3f5-29dd194fcb16"
+          (reference "D1") (unit 1)
+        )
+      )
+    )
+  )
+  (symbol (lib_id "parts:CF12JT220R") (at 153.67 59.69 0) (unit 1)
+    (in_bom yes) (on_board yes) (dnp no) (fields_autoplaced)
+    (property "Reference" "R2" (at 160.02 53.34 0)
+      (effects (font (size 1.524 1.524)))
+    )
+    (property "Value" "CF12JT220R" (at 160.02 55.88 0)
+      (effects (font (size 1.524 1.524)))
+    )
+    (property "Footprint" "parts:STA_CF12_STP" (at 153.67 59.69 0)
+      (effects (font (size 1.27 1.27) italic) hide)
+    )
+    (property "Datasheet" "CF12JT220R" (at 153.67 59.69 0)
+      (effects (font (size 1.27 1.27) italic) hide)
+    )
+    (pin "1")
+    (pin "2")
+    (instances
+      (project "door-sign"
+        (path "/e88230cd-1344-4912-a3f5-29dd194fcb16"
+          (reference "R2") (unit 1)
+        )
+      )
     )
   )
@@
         )
       )
+    )
+  )
+  (symbol (lib_id "parts:CF12JT220R") (at 153.67 46.99 0) (unit 1)
+    (in_bom yes) (on_board yes) (dnp no) (fields_autoplaced)
+    (property "Reference" "R3" (at 160.02 40.64 0)
+      (effects (font (size 1.524 1.524)))
+    )
+    (property "Value" "CF12JT220R" (at 160.02 43.18 0)
+      (effects (font (size 1.524 1.524)))
+    )
+    (property "Footprint" "parts:STA_CF12_STP" (at 153.67 46.99 0)
+      (effects (font (size 1.27 1.27) italic) hide)
+    )
+    (property "Datasheet" "CF12JT220R" (at 153.67 46.99 0)
+      (effects (font (size 1.27 1.27) italic) hide)
+    )
+    (pin "1")
+    (pin "2")
+    (instances
+      (project "door-sign"
+        (path "/e88230cd-1344-4912-a3f5-29dd194fcb16"
+          (reference "R3") (unit 1)
+        )
+      )
+    )
+  )
+  (symbol (lib_id "parts:WP813GD") (at 200.66 99.06 0) (unit 1)
+    (in_bom yes) (on_board yes) (dnp no) (fields_autoplaced)
+    (property "Reference" "D2" (at 199.39 90.17 0)
+      (effects (font (size 1.27 1.27)))
+    )
+    (property "Value" "WP813GD" (at 199.39 92.71 0)
+      (effects (font (size 1.27 1.27)))
+    )
+    (property "Footprint" "parts:LEDRD254W57D1100H1450" (at 200.66 99.06 0)
+      (effects (font (size 1.27 1.27)) (justify bottom) hide)
+    )
+    (property "Datasheet" "" (at 200.66 99.06 0)
+      (effects (font (size 1.27 1.27)) hide)
+    )
+    (property "PARTREV" "V.9B" (at 200.66 99.06 0)
+      (effects (font (size 1.27 1.27)) (justify bottom) hide)
+    )
+    (property "STANDARD" "IPC 7351B" (at 200.66 99.06 0)
+      (effects (font (size 1.27 1.27)) (justify bottom) hide)
+    )
+    (property "SNAPEDA_PACKAGE_ID" "41838" (at 200.66 99.06 0)
+      (effects (font (size 1.27 1.27)) (justify bottom) hide)
+    )
+    (property "MAXIMUM_PACKAGE_HEIGHT" "14.5 mm" (at 200.66 99.06 0)
+      (effects (font (size 1.27 1.27)) (justify bottom) hide)
+    )
+    (property "MANUFACTURER" "Kingbright" (at 200.66 99.06 0)
+      (effects (font (size 1.27 1.27)) (justify bottom) hide)
+    )
+    (pin "1")
+    (pin "2")
+    (instances
+      (project "door-sign"
+        (path "/e88230cd-1344-4912-a3f5-29dd194fcb16"
+          (reference "D2") (unit 1)
+        )
+      )

Commit message: changed design
Parts:
- D1: value WP813GD -> WP813ID
Connections:
- net at BT1.+: now also R1.2
- net at BT1.-: now also D1.1, D2.1
- net at D1.2: now also R2.2
- net at R2.1: now also SW1.1
- net at SW1.2: now also R1.1
- net at SW1.3: now also R3.1
- net at R3.2: now also D2.2
Other:
- moved on the sheet: BT1, D1, D2, R1, R2, R3, SW1
