File: door-sign/door-sign.kicad_pcb (KiCad board)
At the start: 2 copper layers, 100 x 100 mm, 3 parts, among them SW1 200MSP1T1B1M2QEH

Commit message: components done
Parts:
- added D1: WP813GD, parts:LEDRD254W57D1100H1450, F.Cu at (128.7, 40.0)
- added D2: WP813GD, parts:LEDRD254W57D1100H1450, F.Cu at (103.7, 40.0)
- added R2: CF12JT220R, parts:STA_CF12_STP, F.Cu at (92.1, 103.2)
- added R3: CF12JT220R, parts:STA_CF12_STP, F.Cu at (120.9, 103.5)
- moved SW1 24.4 mm to (112.5, 110.0)
- moved R1 18.6 mm to (115.0, 125.0)

Commit message: changed design
Parts:
- D1: value WP813GD -> WP813ID
- moved R2 68.5 mm to (138.4, 52.7), turned to 90 degrees
- moved D2 49.1 mm to (146.7, 63.8), turned to 180 degrees
- moved SW1 42.5 mm to (144.9, 82.5), turned to -90 degrees
- moved R3 36.3 mm to (138.4, 71.8), turned to 90 degrees
- moved R1 30.7 mm to (144.9, 118.1), turned to 0 degrees
- moved BT1 27.3 mm to (106.0, 107.0), turned to 180 degrees
- moved D1 18.6 mm to (146.7, 44.8), turned to 180 degrees
Connections:
- BT1 pad +: unconnected-(BT1-Pad+) -> Net-(BT1-Pad+)
- BT1 pad -: unconnected-(BT1-Pad-) -> Net-(BT1-Pad-)
- D1 pad 1: unconnected-(D1-Pad1) -> Net-(BT1-Pad-)
- D1 pad 2: unconnected-(D1-Pad2) -> Net-(D1-Pad2)
- D2 pad 1: unconnected-(D2-Pad1) -> Net-(BT1-Pad-)
- D2 pad 2: unconnected-(D2-Pad2) -> Net-(D2-Pad2)
- R1 pad 1: unconnected-(R1-Pad1) -> Net-(R1-Pad1)
- R1 pad 2: unconnected-(R1-Pad2) -> Net-(BT1-Pad+)
- R2 pad 1: unconnected-(R2-Pad1) -> Net-(R2-Pad1)
- R2 pad 2: unconnected-(R2-Pad2) -> Net-(D1-Pad2)
- R3 pad 1: unconnected-(R3-Pad1) -> Net-(R3-Pad1)
- R3 pad 2: unconnected-(R3-Pad2) -> Net-(D2-Pad2)
- SW1 pad 1: unconnected-(SW1-Pad1) -> Net-(R2-Pad1)
- SW1 pad 2: unconnected-(SW1-Pad2) -> Net-(R1-Pad1)
- SW1 pad 3: unconnected-(SW1-Pad3) -> Net-(R3-Pad1)
Routing:
- net Net-(BT1-Pad-): track 0.00 -> 133.8 mm
- net Net-(R1-Pad1): track 0.00 -> 42.8 mm
- net Net-(R2-Pad1): track 0.00 -> 40.8 mm
- net Net-(BT1-Pad+): track 0.00 -> 22.2 mm
- net Net-(R3-Pad1): track 0.00 -> 21.1 mm
- net Net-(D1-Pad2): track 0.00 -> 13.9 mm
- net Net-(D2-Pad2): track 0.00 -> 13.9 mm
Other:
- board text added: "Elternampel"
- board text added: "Grün"
- board text added: "Grün | Aus | Rot"
- board text added: "Potentiometer"
- board text added: "Rot"

Commit message: done
Parts:
- added H1: MountingHole, parts:MountingHole_5mm, F.Cu at (71.0, 31.0)
- added H2: MountingHole, parts:MountingHole_5mm, F.Cu at (71.0, 119.0)
- added H3: MountingHole, parts:MountingHole_5mm, F.Cu at (159.0, 31.0)
- added H4: MountingHole, parts:MountingHole_5mm, F.Cu at (159.0, 119.0)
Changed lines of the file:
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@@
   (net 7 "Net-(R2-Pad1)")
   (net 8 "Net-(R3-Pad1)")
+  (footprint "parts:MountingHole_5mm" (layer "F.Cu")
+    (at 71 31)
+    (descr "Mounting Hole 5mm, no annular")
+    (tags "mounting hole 5mm no annular")
+    (property "Sheetfile" "door-sign.kicad_sch")
+    (property "Sheetname" "")
+    (property "ki_description" "Mounting Hole without connection")
+    (property "ki_keywords" "mounting hole")
+    (attr exclude_from_pos_files)
+    (fp_text reference "H1" (at 0 -6) (layer "F.SilkS") hide
+        (effects (font (size 1 1) (thickness 0.15)))
+    )
+    (fp_text value "MountingHole" (at 0 6) (layer "F.Fab") hide
+        (effects (font (size 1 1) (thickness 0.15)))
+    )
+    (fp_text user "${REFERENCE}" (at 0 0) (layer "F.Fab")
+        (effects (font (size 1 1) (thickness 0.15)))
+    )
+    (fp_circle (center 0 0) (end 5 0)
+      (stroke (width 0.15) (type solid)) (fill none) (layer "Cmts.User"))
+    (fp_circle (center 0 0) (end 5.25 0)
+      (stroke (width 0.05) (type solid)) (fill none) (layer "F.CrtYd"))
+    (pad "" np_thru_hole circle (at 0 0) (size 5 5) (drill 5) (layers "*.Cu" "*.Mask"))
+  )
+  (footprint "parts:MountingHole_5mm" (layer "F.Cu")
+    (at 71 119)
+    (descr "Mounting Hole 5mm, no annular")
+    (tags "mounting hole 5mm no annular")
+    (property "Sheetfile" "door-sign.kicad_sch")
+    (property "Sheetname" "")
+    (property "ki_description" "Mounting Hole without connection")
+    (property "ki_keywords" "mounting hole")
+    (attr exclude_from_pos_files)
+    (fp_text reference "H2" (at 0 -6) (layer "F.SilkS") hide
+        (effects (font (size 1 1) (thickness 0.15)))
+    )
+    (fp_text value "MountingHole" (at 0 6) (layer "F.Fab") hide
+        (effects (font (size 1 1) (thickness 0.15)))
+    )
+    (fp_text user "${REFERENCE}" (at 0 0) (layer "F.Fab")
+        (effects (font (size 1 1) (thickness 0.15)))
+    )
+    (fp_circle (center 0 0) (end 5 0)
+      (stroke (width 0.15) (type solid)) (fill none) (layer "Cmts.User"))
+    (fp_circle (center 0 0) (end 5.25 0)
+      (stroke (width 0.05) (type solid)) (fill none) (layer "F.CrtYd"))
+    (pad "" np_thru_hole circle (at 0 0) (size 5 5) (drill 5) (layers "*.Cu" "*.Mask"))
+  )
+  (footprint "parts:MountingHole_5mm" (layer "F.Cu")
+    (at 159 31)
+    (descr "Mounting Hole 5mm, no annular")
+    (tags "mounting hole 5mm no annular")
+    (property "Sheetfile" "door-sign.kicad_sch")
+    (property "Sheetname" "")
+    (property "ki_description" "Mounting Hole without connection")
+    (property "ki_keywords" "mounting hole")
+    (attr exclude_from_pos_files)
+    (fp_text reference "H3" (at 0 -6) (layer "F.SilkS") hide
+        (effects (font (size 1 1) (thickness 0.15)))
+    )
+    (fp_text value "MountingHole" (at 0 6) (layer "F.Fab") hide
+        (effects (font (size 1 1) (thickness 0.15)))
+    )
+    (fp_text user "${REFERENCE}" (at 0 0) (layer "F.Fab")
+        (effects (font (size 1 1) (thickness 0.15)))
+    )
+    (fp_circle (center 0 0) (end 5 0)
+      (stroke (width 0.15) (type solid)) (fill none) (layer "Cmts.User"))
+    (fp_circle (center 0 0) (end 5.25 0)
+      (stroke (width 0.05) (type solid)) (fill none) (layer "F.CrtYd"))
+    (pad "" np_thru_hole circle (at 0 0) (size 5 5) (drill 5) (layers "*.Cu" "*.Mask"))
+  )
   (footprint "parts:STA_CF12_STP" (layer "F.Cu")
     (at 138.42 71.75 90)
@@
       (stroke (width 0.0254) (type solid)) (layer "F.Fab"))
     (pad "1" thru_hole rect (at 0 0 90) (size 1.524 1.524) (drill 1.016) (layers "*.Cu" "*.Mask")
-      (net 8 "Net-(R3-Pad1)") (pintype "unspecified"))
+      (net 8 "Net-(R3-Pad1)") (pintype "passive"))
     (pad "2" thru_hole circle (at 15.748 0 90) (size 1.524 1.524) (drill 1.016) (layers "*.Cu" "*.Mask")
-      (net 4 "Net-(D2-Pad2)") (pintype "unspecified"))
+      (net 4 "Net-(D2-Pad2)") (pintype "passive"))
     (model "/Users/chao/git/Door-sign/libs/STA_CF12_STP.step"
       (offset (xyz 0 0 0))
@@
       (net 1 "Net-(BT1-Pad+)") (pintype "passive") (solder_mask_margin 0.102))
     (pad "3" thru_hole circle (at 2.54 2.87) (size 1.16 1.16) (drill 0.76) (layers "*.Cu" "*.Mask")
-      (net 5 "unconnected-(R1-Pad3)") (pintype "passive") (solder_mask_margin 0.102))
+      (net 5 "unconnected-(R1-Pad3)") (pintype "passive+no_connect") (solder_mask_margin 0.102))
     (model "/Users/chao/git/Door-sign/libs/3352T-1-501LF.step"
       (offset (xyz 0 0 0))
@@
       (rotate (xyz -90 0 0))
     )
+  )
+  (footprint "parts:MountingHole_5mm" (layer "F.Cu")
+    (at 159 119)
+    (descr "Mounting Hole 5mm, no annular")
+    (tags "mounting hole 5mm no annular")
+    (property "Sheetfile" "door-sign.kicad_sch")
+    (property "Sheetname" "")
+    (property "ki_description" "Mounting Hole without connection")
+    (property "ki_keywords" "mounting hole")
+    (attr exclude_from_pos_files)
+    (fp_text reference "H4" (at 0 -6) (layer "F.SilkS") hide
+        (effects (font (size 1 1) (thickness 0.15)))
+    )
+    (fp_text value "MountingHole" (at 0 6) (layer "F.Fab") hide
+        (effects (font (size 1 1) (thickness 0.15)))
+    )
+    (fp_text user "${REFERENCE}" (at 0 0) (layer "F.Fab")
+        (effects (font (size 1 1) (thickness 0.15)))
+    )
+    (fp_circle (center 0 0) (end 5 0)
+      (stroke (width 0.15) (type solid)) (fill none) (layer "Cmts.User"))
+    (fp_circle (center 0 0) (end 5.25 0)
+      (stroke (width 0.05) (type solid)) (fill none) (layer "F.CrtYd"))
+    (pad "" np_thru_hole circle (at 0 0) (size 5 5) (drill 5) (layers "*.Cu" "*.Mask"))
   )
   (footprint "parts:200MSP1T1B1M2QEH_EWI" (layer "F.Cu")
@@
       (stroke (width 0.508) (type solid)) (fill none) (layer "F.Fab"))
     (pad "1" thru_hole circle (at 0 0 270) (size 1.6002 1.6002) (drill 1.0922) (layers "*.Cu" "*.Mask")
-      (net 7 "Net-(R2-Pad1)") (pinfunction "1") (pintype "unspecified"))
+      (net 7 "Net-(R2-Pad1)") (pinfunction "1") (pintype "passive"))
     (pad "2" thru_hole circle (at 2.54 0 270) (size 1.6002 1.6002) (drill 1.0922) (layers "*.Cu" "*.Mask")
-      (net 6 "Net-(R1-Pad1)") (pinfunction "2") (pintype "unspecified"))
+      (net 6 "Net-(R1-Pad1)") (pinfunction "2") (pintype "passive"))
     (pad "3" thru_hole circle (at 5.08 0 270) (size 1.6002 1.6002) (drill 1.0922) (layers "*.Cu" "*.Mask")
-      (net 8 "Net-(R3-Pad1)") (pinfunction "3") (pintype "unspecified"))
+      (net 8 "Net-(R3-Pad1)") (pinfunction "3") (pintype "passive"))
     (model "/Users/chao/git/Door-sign/libs/200MSP1T1B1M2QEH.STEP"
       (offset (xyz 2.5 0 0))
@@
       (stroke (width 0.0254) (type solid)) (layer "F.Fab"))
     (pad "1" thru_hole rect (at 0 0 90) (size 1.524 1.524) (drill 1.016) (layers "*.Cu" "*.Mask")
-      (net 7 "Net-(R2-Pad1)") (pintype "unspecified"))
+      (net 7 "Net-(R2-Pad1)") (pintype "passive"))
     (pad "2" thru_hole circle (at 15.748 0 90) (size 1.524 1.524) (drill 1.016) (layers "*.Cu" "*.Mask")
-      (net 3 "Net-(D1-Pad2)") (pintype "unspecified"))
+      (net 3 "Net-(D1-Pad2)") (pintype "passive"))
     (model "/Users/chao/git/Door-sign/libs/STA_CF12_STP.step"
       (offset (xyz 0 0 0))

Commit message: moved parts a little bit
Parts:
- moved R1 3.32 mm to (148.2, 118.5)
- moved D1 3.32 mm to (150.0, 45.1)
- moved R2 3.32 mm to (141.7, 53.1)
- moved D2 3.32 mm to (150.0, 64.1)
- moved R3 3.32 mm to (141.7, 72.1)
- moved SW1 3.32 mm to (148.2, 82.8)
Routing:
- net Net-(BT1-Pad-): track 133.8 -> 136.9 mm
- net Net-(BT1-Pad+): track 22.2 -> 25.4 mm
Changed lines of the file:
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@@
   )
   (footprint "parts:STA_CF12_STP" (layer "F.Cu")
-    (at 138.42 71.75 90)
+    (at 141.72 72.07 90)
     (tags "CF12JT220R ")
     (property "Sheetfile" "door-sign.kicad_sch")
@@
   )
   (footprint "parts:LEDRD254W57D1100H1450" (layer "F.Cu")
-    (at 146.67 63.75 180)
+    (at 149.97 64.07 180)
     (property "MANUFACTURER" "Kingbright")
     (property "MAXIMUM_PACKAGE_HEIGHT" "14.5 mm")
@@
   )
   (footprint "parts:LEDRD254W57D1100H1450" (layer "F.Cu")
-    (at 146.67 44.75 180)
+    (at 149.97 45.07 180)
     (property "MANUFACTURER" "Kingbright")
     (property "MAXIMUM_PACKAGE_HEIGHT" "14.5 mm")
@@
   )
   (footprint "parts:TRIM_3352T-1-501LF" (layer "F.Cu")
-    (at 144.92 118.13)
+    (at 148.22 118.45)
     (property "MANUFACTURER" "Bourns")
     (property "MAXIMUM_PACKAGE_HEIGHT" "4.32mm")
@@
   )
   (footprint "parts:200MSP1T1B1M2QEH_EWI" (layer "F.Cu")
-    (at 144.92 82.5 -90)
+    (at 148.22 82.82 -90)
     (tags "200MSP1T1B1M2QEH ")
     (property "Sheetfile" "door-sign.kicad_sch")
@@
   )
   (footprint "parts:STA_CF12_STP" (layer "F.Cu")
-    (at 138.42 52.748 90)
+    (at 141.72 53.068 90)
     (tags "CF12JT220R ")
     (property "Sheetfile" "door-sign.kicad_sch")
@@
     )
   )
-  (gr_rect (start 141 74) (end 148.62 122.26)
+  (gr_rect (start 144.3 74.32) (end 151.92 122.58)
     (stroke (width 0.15) (type default)) (fill none) (layer "F.SilkS"))
-  (gr_rect (start 135.92 33.36) (end 153.7 74)
+  (gr_rect (start 139.22 33.68) (end 157 74.32)
     (stroke (width 0.15) (type default)) (fill none) (layer "F.SilkS"))
   (gr_line (start 70 125) (end 160 125)
@@
   (gr_arc (start 65 30) (mid 66.464466 26.464466) (end 70 25)
     (stroke (width 0.1) (type default)) (layer "Edge.Cuts"))
-  (gr_text "Rot" (at 146.8 47) (layer "F.SilkS")
+  (gr_text "Rot" (at 150.1 47.32) (layer "F.SilkS")
     (effects (font (size 1 1) (thickness 0.15)))
   )
-  (gr_text "Potentiometer" (at 145.02 107.9 90) (layer "F.SilkS")
+  (gr_text "Potentiometer" (at 148.32 108.22 90) (layer "F.SilkS")
     (effects (font (size 1 1) (thickness 0.15)))
   )
-  (gr_text "Grün" (at 146.6 66.2) (layer "F.SilkS")
+  (gr_text "Grün" (at 149.9 66.52) (layer "F.SilkS")
     (effects (font (size 1 1) (thickness 0.15)))
   )
-  (gr_text "Grün | Aus | Rot" (at 139.62 85 90) (layer "F.SilkS")
+  (gr_text "Grün | Aus | Rot" (at 142.92 85.32 90) (layer "F.SilkS")
     (effects (font (size 1 1) (thickness 0.15)))
   )
@@
   )
   (segment (start 132.16 113.64) (end 132.16 121.36) (width 0.6) (layer "B.Cu") (net 1))
-  (segment (start 143.8 122.8) (end 144.92 121.68) (width 0.6) (layer "B.Cu") (net 1))
-  (segment (start 133.6 122.8) (end 143.8 122.8) (width 0.6) (layer "B.Cu") (net 1))
   (segment (start 132.16 121.36) (end 133.6 122.8) (width 0.6) (layer "B.Cu") (net 1))
-  (segment (start 144.92 121.68) (end 144.92 121) (width 0.6) (layer "B.Cu") (net 1))
-  (segment (start 152.2 47) (end 149.95 44.75) (width 0.6) (layer "B.Cu") (net 2))
-  (segment (start 149.4 124) (end 152.2 121.2) (width 0.6) (layer "B.Cu") (net 2))
+  (segment (start 148.11 122.11) (end 148.22 122) (width 0.6) (layer "B.Cu") (net 1))
+  (segment (start 147.42 122.8) (end 148.11 122.11) (width 0.6) (layer "B.Cu") (net 1))
+  (segment (start 133.6 122.8) (end 147.42 122.8) (width 0.6) (layer "B.Cu") (net 1))
+  (segment (start 148.22 122) (end 148.22 121.32) (width 0.6) (layer "B.Cu") (net 1))
+  (segment (start 132 124) (end 153 124) (width 0.6) (layer "B.Cu") (net 2))
+  (segment (start 155.5 47.32) (end 153.25 45.07) (width 0.6) (layer "B.Cu") (net 2))
+  (segment (start 155.5 66.12) (end 155.5 68.52) (width 0.6) (layer "B.Cu") (net 2))
+  (segment (start 153.25 45.07) (end 151.24 45.07) (width 0.6) (layer "B.Cu") (net 2))
+  (segment (start 151.24 64.07) (end 153.45 64.07) (width 0.6) (layer "B.Cu") (net 2))
+  (segment (start 153.01 124.01) (end 155.5 121.52) (width 0.6) (layer "B.Cu") (net 2))
+  (segment (start 153.45 64.07) (end 155.5 66.12) (width 0.6) (layer "B.Cu") (net 2))
+  (segment (start 130.2 102.01) (end 130.2 122.2) (width 0.6) (layer "B.Cu") (net 2))
+  (segment (start 130.2 122.2) (end 132 124) (width 0.6) (layer "B.Cu") (net 2))
   (segment (start 132.16 100.05) (end 130.2 102.01) (width 0.6) (layer "B.Cu") (net 2))
-  (segment (start 152.2 65.8) (end 152.2 68.2) (width 0.6) (layer "B.Cu") (net 2))
-  (segment (start 149.95 44.75) (end 147.94 44.75) (width 0.6) (layer "B.Cu") (net 2))
-  (segment (start 147.94 63.75) (end 150.15 63.75) (width 0.6) (layer "B.Cu") (net 2))
-  (segment (start 130.2 102.01) (end 130.2 122.2) (width 0.6) (layer "B.Cu") (net 2))
-  (segment (start 150.15 63.75) (end 152.2 65.8) (width 0.6) (layer "B.Cu") (net 2))
-  (segment (start 130.2 122.2) (end 132 124) (width 0.6) (layer "B.Cu") (net 2))
-  (segment (start 132 124) (end 149.4 124) (width 0.6) (layer "B.Cu") (net 2))
-  (segment (start 152.2 121.2) (end 152.2 68.2) (width 0.6) (layer "B.Cu") (net 2))
-  (segment (start 152.2 68.2) (end 152.2 47) (width 0.6) (layer "B.Cu") (net 2))
-  (segment (start 145.4 38.4) (end 145.4 44.75) (width 0.6) (layer "B.Cu") (net 3))
-  (segment (start 144 37) (end 145.4 38.4) (width 0.6) (layer "B.Cu") (net 3))
-  (segment (start 138.42 37) (end 144 37) (width 0.6) (layer "B.Cu") (net 3))
-  (segment (start 145.4 57.4) (end 145.4 63.75) (width 0.6) (layer "B.Cu") (net 4))
-  (segment (start 138.42 56.002) (end 144.002 56.002) (width 0.6) (layer "B.Cu") (net 4))
-  (segment (start 144.002 56.002) (end 145.4 57.4) (width 0.6) (layer "B.Cu") (net 4))
-  (segment (start 147.84 85.04) (end 144.92 85.04) (width 0.6) (layer "B.Cu") (net 6))
-  (segment (start 142.38 119.72) (end 149.8 112.3) (width 0.6) (layer "B.Cu") (net 6))
-  (segment (start 142.38 121) (end 142.38 119.72) (width 0.6) (layer "B.Cu") (net 6))
-  (segment (start 149.8 112.3) (end 149.8 87) (width 0.6) (layer "B.Cu") (net 6))
-  (segment (start 149.8 87) (end 147.84 85.04) (width 0.6) (layer "B.Cu") (net 6))
-  (segment (start 134.8 64.6) (end 134.8 54) (width 0.6) (layer "B.Cu") (net 7))
-  (segment (start 136.052 52.748) (end 138.42 52.748) (width 0.6) (layer "B.Cu") (net 7))
-  (segment (start 144.92 67.92) (end 143 66) (width 0.6) (layer "B.Cu") (net 7))
-  (segment (start 136.2 66) (end 134.8 64.6) (width 0.6) (layer "B.Cu") (net 7))
-  (segment (start 143 66) (end 136.2 66) (width 0.6) (layer "B.Cu") (net 7))
-  (segment (start 134.8 54) (end 136.052 52.748) (width 0.6) (layer "B.Cu") (net 7))
-  (segment (start 144.92 82.5) (end 144.92 67.92) (width 0.6) (layer "B.Cu") (net 7))
-  (segment (start 140.58 87.58) (end 144.92 87.58) (width 0.6) (layer "B.Cu") (net 8))
-  (segment (start 138.42 85.42) (end 140.58 87.58) (width 0.6) (layer "B.Cu") (net 8))
-  (segment (start 138.42 71.75) (end 138.42 85.42) (width 0.6) (layer "B.Cu") (net 8))
+  (segment (start 155.5 121.52) (end 155.5 68.52) (width 0.6) (layer "B.Cu") (net 2))
+  (segment (start 155.5 68.52) (end 155.5 47.32) (width 0.6) (layer "B.Cu") (net 2))
+  (segment (start 153 124) (end 153.01 124.01) (width 0.6) (layer "B.Cu") (net 2))
+  (segment (start 148.7 38.72) (end 148.7 45.07) (width 0.6) (layer "B.Cu") (net 3))
+  (segment (start 147.3 37.32) (end 148.7 38.72) (width 0.6) (layer "B.Cu") (net 3))
+  (segment (start 141.72 37.32) (end 147.3 37.32) (width 0.6) (layer "B.Cu") (net 3))
+  (segment (start 148.7 57.72) (end 148.7 64.07) (width 0.6) (layer "B.Cu") (net 4))
+  (segment (start 141.72 56.322) (end 147.302 56.322) (width 0.6) (layer "B.Cu") (net 4))
+  (segment (start 147.302 56.322) (end 148.7 57.72) (width 0.6) (layer "B.Cu") (net 4))
+  (segment (start 151.14 85.36) (end 148.22 85.36) (width 0.6) (layer "B.Cu") (net 6))
+  (segment (start 145.68 120.04) (end 153.1 112.62) (width 0.6) (layer "B.Cu") (net 6))
+  (segment (start 145.68 121.32) (end 145.68 120.04) (width 0.6) (layer "B.Cu") (net 6))
+  (segment (start 153.1 112.62) (end 153.1 87.32) (width 0.6) (layer "B.Cu") (net 6))
+  (segment (start 153.1 87.32) (end 151.14 85.36) (width 0.6) (layer "B.Cu") (net 6))
+  (segment (start 138.1 64.92) (end 138.1 54.32) (width 0.6) (layer "B.Cu") (net 7))
+  (segment (start 139.352 53.068) (end 141.72 53.068) (width 0.6) (layer "B.Cu") (net 7))
+  (segment (start 148.22 68.24) (end 146.3 66.32) (width 0.6) (layer "B.Cu") (net 7))
+  (segment (start 139.5 66.32) (end 138.1 64.92) (width 0.6) (layer "B.Cu") (net 7))
+  (segment (start 146.3 66.32) (end 139.5 66.32) (width 0.6) (layer "B.Cu") (net 7))
+  (segment (start 138.1 54.32) (end 139.352 53.068) (width 0.6) (layer "B.Cu") (net 7))
+  (segment (start 148.22 82.82) (end 148.22 68.24) (width 0.6) (layer "B.Cu") (net 7))
+  (segment (start 143.88 87.9) (end 148.22 87.9) (width 0.6) (layer "B.Cu") (net 8))
+  (segment (start 141.72 85.74) (end 143.88 87.9) (width 0.6) (layer "B.Cu") (net 8))
+  (segment (start 141.72 72.07) (end 141.72 85.74) (width 0.6) (layer "B.Cu") (net 8))
 )

Commit message: update component values
Parts:
- R1: value 3352T-1-501LF -> 3352T-1-201LF
- R2, R3: value CF12JT220R -> CF12JT110R
Changed lines of the file:
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@@
       (outputformat 1)
       (mirror false)
-      (drillshape 1)
+      (drillshape 0)
       (scaleselection 1)
-      (outputdirectory "")
+      (outputdirectory "gerber/")
     )
   )
@@
         (effects (font (size 1 1) (thickness 0.15)))
     )
-    (fp_text value "CF12JT220R" (at 7.874 0 90 unlocked) (layer "F.Fab") hide
+    (fp_text value "CF12JT110R" (at 7.874 0 90 unlocked) (layer "F.Fab") hide
         (effects (font (size 1 1) (thickness 0.15)))
     )
@@
         (effects (font (size 1 1) (thickness 0.15)))
     )
-    (fp_text value "3352T-1-501LF" (at 7.63 6.065) (layer "F.Fab") hide
+    (fp_text value "3352T-1-201LF" (at 7.63 6.065) (layer "F.Fab") hide
         (effects (font (size 1 1) (thickness 0.15)))
     )
@@
         (effects (font (size 1 1) (thickness 0.15)))
     )
-    (fp_text value "CF12JT220R" (at 7.874 0 90 unlocked) (layer "F.Fab") hide
-        (effects (font (size 1 1) (thickness 0.15)))
-    )
+    (fp_text value "CF12JT110R" (at 7.874 0 90 unlocked) (layer "F.Fab") hide
+        (effects (font (size 1 1) (thickness 0.15)))
+    )
