File: door-sign/door-sign.kicad_pcb (KiCad board)
At the start: 2 copper layers, 100 x 100 mm, 11 parts, among them SW1 200MSP1T1B1M2QEH

Commit message: fixed errors
Parts:
- moved R1 0.10 mm to (148.1, 118.5)
Connections:
- SW1 pad 1: Net-(R2-Pad1) -> Net-(R3-Pad1)
- SW1 pad 3: Net-(R3-Pad1) -> Net-(R2-Pad1)
Routing:
- net Net-(R2-Pad1): track 40.8 -> 51.9 mm
- net Net-(R3-Pad1): track 21.1 -> 15.2 mm
- net Net-(R1-Pad1): track 42.8 -> 38.0 mm
Other:
- board text added: "Version 1.0 2024.03.26"
Changed lines of the file:
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@@
   )
   (footprint "parts:TRIM_3352T-1-501LF" (layer "F.Cu")
-    (at 148.22 118.45)
+    (at 148.115 118.45)
     (property "MANUFACTURER" "Bourns")
     (property "MAXIMUM_PACKAGE_HEIGHT" "4.32mm")
@@
       (stroke (width 0.508) (type solid)) (fill none) (layer "F.Fab"))
     (pad "1" thru_hole circle (at 0 0 270) (size 1.6002 1.6002) (drill 1.0922) (layers "*.Cu" "*.Mask")
-      (net 7 "Net-(R2-Pad1)") (pinfunction "1") (pintype "passive"))
+      (net 8 "Net-(R3-Pad1)") (pinfunction "1") (pintype "passive"))
     (pad "2" thru_hole circle (at 2.54 0 270) (size 1.6002 1.6002) (drill 1.0922) (layers "*.Cu" "*.Mask")
       (net 6 "Net-(R1-Pad1)") (pinfunction "2") (pintype "passive"))
     (pad "3" thru_hole circle (at 5.08 0 270) (size 1.6002 1.6002) (drill 1.0922) (layers "*.Cu" "*.Mask")
-      (net 8 "Net-(R3-Pad1)") (pinfunction "3") (pintype "passive"))
+      (net 7 "Net-(R2-Pad1)") (pinfunction "3") (pintype "passive"))
     (model "/Users/chao/git/Door-sign/libs/200MSP1T1B1M2QEH.STEP"
       (offset (xyz 2.5 0 0))
@@
   (gr_arc (start 65 30) (mid 66.464466 26.464466) (end 70 25)
     (stroke (width 0.1) (type default)) (layer "Edge.Cuts"))
+  (gr_text "Version 1.0\n2024.03.26" (at 82.1 94.2) (layer "F.SilkS")
+    (effects (font (size 1 1) (thickness 0.15)))
+  )
   (gr_text "Rot" (at 150.1 47.32) (layer "F.SilkS")
     (effects (font (size 1 1) (thickness 0.15)))
@@
     (effects (font (size 6.5 6.5) (thickness 1.4) bold) (justify left bottom))
   )
+  (segment (start 147.5 122.8) (end 148.115 122.185) (width 0.6) (layer "B.Cu") (net 1))
   (segment (start 132.16 113.64) (end 132.16 121.36) (width 0.6) (layer "B.Cu") (net 1))
+  (segment (start 133.6 122.8) (end 147.5 122.8) (width 0.6) (layer "B.Cu") (net 1))
   (segment (start 132.16 121.36) (end 133.6 122.8) (width 0.6) (layer "B.Cu") (net 1))
-  (segment (start 148.11 122.11) (end 148.22 122) (width 0.6) (layer "B.Cu") (net 1))
-  (segment (start 147.42 122.8) (end 148.11 122.11) (width 0.6) (layer "B.Cu") (net 1))
-  (segment (start 133.6 122.8) (end 147.42 122.8) (width 0.6) (layer "B.Cu") (net 1))
-  (segment (start 148.22 122) (end 148.22 121.32) (width 0.6) (layer "B.Cu") (net 1))
+  (segment (start 148.115 122.185) (end 148.115 121.32) (width 0.6) (layer "B.Cu") (net 1))
   (segment (start 132 124) (end 153 124) (width 0.6) (layer "B.Cu") (net 2))
   (segment (start 155.5 47.32) (end 153.25 45.07) (width 0.6) (layer "B.Cu") (net 2))
@@
   (segment (start 141.72 56.322) (end 147.302 56.322) (width 0.6) (layer "B.Cu") (net 4))
   (segment (start 147.302 56.322) (end 148.7 57.72) (width 0.6) (layer "B.Cu") (net 4))
-  (segment (start 151.14 85.36) (end 148.22 85.36) (width 0.6) (layer "B.Cu") (net 6))
-  (segment (start 145.68 120.04) (end 153.1 112.62) (width 0.6) (layer "B.Cu") (net 6))
-  (segment (start 145.68 121.32) (end 145.68 120.04) (width 0.6) (layer "B.Cu") (net 6))
-  (segment (start 153.1 112.62) (end 153.1 87.32) (width 0.6) (layer "B.Cu") (net 6))
-  (segment (start 153.1 87.32) (end 151.14 85.36) (width 0.6) (layer "B.Cu") (net 6))
+  (segment (start 145.575 86.425) (end 146.64 85.36) (width 0.6) (layer "B.Cu") (net 6))
+  (segment (start 146.64 85.36) (end 148.22 85.36) (width 0.6) (layer "B.Cu") (net 6))
+  (segment (start 145.575 121.32) (end 145.575 86.425) (width 0.6) (layer "B.Cu") (net 6))
+  (segment (start 140.18 67) (end 138.1 64.92) (width 0.6) (layer "B.Cu") (net 7))
+  (segment (start 152 69) (end 150 67) (width 0.6) (layer "B.Cu") (net 7))
+  (segment (start 148.22 87.9) (end 150.1 87.9) (width 0.6) (layer "B.Cu") (net 7))
+  (segment (start 152 86) (end 152 69) (width 0.6) (layer "B.Cu") (net 7))
+  (segment (start 150 67) (end 140.18 67) (width 0.6) (layer "B.Cu") (net 7))
+  (segment (start 139.352 53.068) (end 141.72 53.068) (width 0.6) (layer "B.Cu") (net 7))
+  (segment (start 150.1 87.9) (end 152 86) (width 0.6) (layer "B.Cu") (net 7))
+  (segment (start 138.1 54.32) (end 139.352 53.068) (width 0.6) (layer "B.Cu") (net 7))
   (segment (start 138.1 64.92) (end 138.1 54.32) (width 0.6) (layer "B.Cu") (net 7))
-  (segment (start 139.352 53.068) (end 141.72 53.068) (width 0.6) (layer "B.Cu") (net 7))
-  (segment (start 148.22 68.24) (end 146.3 66.32) (width 0.6) (layer "B.Cu") (net 7))
-  (segment (start 139.5 66.32) (end 138.1 64.92) (width 0.6) (layer "B.Cu") (net 7))
-  (segment (start 146.3 66.32) (end 139.5 66.32) (width 0.6) (layer "B.Cu") (net 7))
-  (segment (start 138.1 54.32) (end 139.352 53.068) (width 0.6) (layer "B.Cu") (net 7))
-  (segment (start 148.22 82.82) (end 148.22 68.24) (width 0.6) (layer "B.Cu") (net 7))
-  (segment (start 143.88 87.9) (end 148.22 87.9) (width 0.6) (layer "B.Cu") (net 8))
-  (segment (start 141.72 85.74) (end 143.88 87.9) (width 0.6) (layer "B.Cu") (net 8))
-  (segment (start 141.72 72.07) (end 141.72 85.74) (width 0.6) (layer "B.Cu") (net 8))
+  (segment (start 148.22 78.22) (end 148.22 82.82) (width 0.6) (layer "B.Cu") (net 8))
+  (segment (start 147 77) (end 148.22 78.22) (width 0.6) (layer "B.Cu") (net 8))
+  (segment (start 141.72 74.72) (end 144 77) (width 0.6) (layer "B.Cu") (net 8))
+  (segment (start 144 77) (end 147 77) (width 0.6) (layer "B.Cu") (net 8))
+  (segment (start 141.72 72.07) (end 141.72 74.72) (width 0.6) (layer "B.Cu") (net 8))
 )
